File: kapula/kapula.sch (KiCad schematic (older format))
At the start: 71 parts, among them J1 Conn_Coaxial, J2 Display, Q1 BC847, SW1 SW_SPST, SW2 Rotary_Encoder_Switch, T1 Transformer_SP_1S, U1 MCP73831-2-OT, U2 MIC5501-3.0YM5, U3 EFR32FG14P233F256GM48-B, X1 38.4 MHz TCXO

Commit message: PCB: Add some components and footprints
Parts:
- added C18, C26, C27, C38, C39: 1n, Capacitor_SMD:C_0603_1608Metric_Pad1.05x0.95mm_HandSolder, symbol Device:C
- added C28: 0, Capacitor_SMD:C_0603_1608Metric_Pad1.05x0.95mm_HandSolder, symbol Device:C
- added C29: TBD, Capacitor_SMD:C_0603_1608Metric_Pad1.05x0.95mm_HandSolder, symbol Device:C
- added FB1: Ferrite_Bead, Inductor_SMD:L_0603_1608Metric_Pad1.05x0.95mm_HandSolder, symbol Device:Ferrite_Bead
- added J1, J3: SMA, Connector_Coaxial:SMA_Amphenol_901-144_Vertical, symbol Connector:Conn_Coaxial
- added L10, L11, L6: TBD, Inductor_SMD:L_0603_1608Metric_Pad1.05x0.95mm_HandSolder, symbol Device:L
- added R2, R4, R7, R8: 0, Resistor_SMD:R_0603_1608Metric_Pad1.05x0.95mm_HandSolder, symbol Device:R
- added R3, R5: 1k, Resistor_SMD:R_0603_1608Metric_Pad1.05x0.95mm_HandSolder, symbol Device:R
- added SW3: SW_Push, symbol Switch:SW_Push
- added T1: ETC4-1-2TR, kapula:ETC4-1-2TR, symbol Device:Transformer_SP_1S
- added U4: AS213-92LF, Package_TO_SOT_SMD:SOT-363_SC-70-6, symbol kapula:SKY13270-92LF
- C1, C10, C11, C12, C13, C14, C15, C16, C17, C2, C20, C3, C4, C5, C6, C7, C8, C9: footprint Capacitor_SMD:C_0603_1608Metric -> Capacitor_SMD:C_0603_1608Metric_Pad1.05x0.95mm_HandSolder
- C19: renamed from C18; footprint Capacitor_SMD:C_0603_1608Metric -> Capacitor_SMD:C_0603_1608Metric_Pad1.05x0.95mm_HandSolder
- C21: renamed from C19; value TBD -> 0; footprint Capacitor_SMD:C_0603_1608Metric -> Capacitor_SMD:C_0603_1608Metric_Pad1.05x0.95mm_HandSolder; DNP (none) -> DNP
- C22: value TBD -> 1n; footprint Capacitor_SMD:C_0603_1608Metric -> Capacitor_SMD:C_0603_1608Metric_Pad1.05x0.95mm_HandSolder
- C23: renamed from C21; footprint Capacitor_SMD:C_0603_1608Metric -> Capacitor_SMD:C_0603_1608Metric_Pad1.05x0.95mm_HandSolder
- C24: renamed from C23; footprint Capacitor_SMD:C_0603_1608Metric -> Capacitor_SMD:C_0603_1608Metric_Pad1.05x0.95mm_HandSolder
- C25: renamed from C24; footprint Capacitor_SMD:C_0603_1608Metric -> Capacitor_SMD:C_0603_1608Metric_Pad1.05x0.95mm_HandSolder
- C30: renamed from C27; footprint Capacitor_SMD:C_0603_1608Metric -> Capacitor_SMD:C_0603_1608Metric_Pad1.05x0.95mm_HandSolder
- C31: renamed from C29; footprint Capacitor_SMD:C_0603_1608Metric -> Capacitor_SMD:C_0603_1608Metric_Pad1.05x0.95mm_HandSolder
- C32: renamed from C30; footprint Capacitor_SMD:C_0603_1608Metric -> Capacitor_SMD:C_0603_1608Metric_Pad1.05x0.95mm_HandSolder
- C33: renamed from C31; footprint Capacitor_SMD:C_0603_1608Metric -> Capacitor_SMD:C_0603_1608Metric_Pad1.05x0.95mm_HandSolder
- C34: renamed from C32; footprint Capacitor_SMD:C_0603_1608Metric -> Capacitor_SMD:C_0603_1608Metric_Pad1.05x0.95mm_HandSolder
- C35: renamed from C25; footprint Capacitor_SMD:C_0603_1608Metric -> Capacitor_SMD:C_0603_1608Metric_Pad1.05x0.95mm_HandSolder
- C36: renamed from C26; footprint Capacitor_SMD:C_0603_1608Metric -> Capacitor_SMD:C_0603_1608Metric_Pad1.05x0.95mm_HandSolder
- C37: renamed from C28; footprint Capacitor_SMD:C_0603_1608Metric -> Capacitor_SMD:C_0603_1608Metric_Pad1.05x0.95mm_HandSolder
- C40: renamed from C33; footprint Capacitor_SMD:C_0603_1608Metric -> Capacitor_SMD:C_0603_1608Metric_Pad1.05x0.95mm_HandSolder
- F1: footprint Resistor_SMD:R_1206_3216Metric -> Resistor_SMD:R_1206_3216Metric_Pad1.42x1.75mm_HandSolder
- FB2: renamed from FB1; footprint Inductor_SMD:L_0603_1608Metric -> Inductor_SMD:L_0603_1608Metric_Pad1.05x0.95mm_HandSolder
- J2: renamed from J1; value Conn_Coaxial -> SMA
- L2, L3, L4, L5: footprint Inductor_SMD:L_0603_1608Metric -> Inductor_SMD:L_0603_1608Metric_Pad1.05x0.95mm_HandSolder
- L7: renamed from L6; footprint Inductor_SMD:L_0603_1608Metric -> Inductor_SMD:L_0603_1608Metric_Pad1.05x0.95mm_HandSolder
- L8: renamed from L7; footprint Inductor_SMD:L_0603_1608Metric -> Inductor_SMD:L_0603_1608Metric_Pad1.05x0.95mm_HandSolder
- L9: renamed from L8; footprint Inductor_SMD:L_0603_1608Metric -> Inductor_SMD:L_0603_1608Metric_Pad1.05x0.95mm_HandSolder
- Q1: footprint Package_TO_SOT_SMD:SOT-23 -> Package_TO_SOT_SMD:SOT-23_Handsoldering
- R1, R6: footprint Resistor_SMD:R_0603_1608Metric -> Resistor_SMD:R_0603_1608Metric_Pad1.05x0.95mm_HandSolder
- R10: renamed from R3; footprint Resistor_SMD:R_0603_1608Metric -> Resistor_SMD:R_0603_1608Metric_Pad1.05x0.95mm_HandSolder
- R11: renamed from R4; footprint Resistor_SMD:R_0603_1608Metric -> Resistor_SMD:R_0603_1608Metric_Pad1.05x0.95mm_HandSolder
- R12: renamed from R5; footprint Resistor_SMD:R_0603_1608Metric -> Resistor_SMD:R_0603_1608Metric_Pad1.05x0.95mm_HandSolder
- R9: renamed from R2; footprint Resistor_SMD:R_0603_1608Metric -> Resistor_SMD:R_0603_1608Metric_Pad1.05x0.95mm_HandSolder
- SW2: value Rotary_Encoder_Switch -> EC11B15242B1; footprint Rotary_Encoder:RotaryEncoder_Alps_EC11E-Switch_Vertical_H20mm_CircularMountingHoles -> kapula:RotaryEncoder_Alps_EC11B-Switch_Horizontal
- T2: renamed from T1; value Transformer_SP_1S -> ETC4-1-2TR; footprint (none) -> kapula:ETC4-1-2TR
- U1, U2: footprint Package_TO_SOT_SMD:SOT-23-5 -> Package_TO_SOT_SMD:SOT-23-5_HandSoldering
- X1: value 38.4 MHz TCXO -> TCO22384001805; footprint Oscillator:Oscillator_SMD_EuroQuartz_XO32-4Pin_3.2x2.5mm -> Oscillator:Oscillator_SMD_EuroQuartz_XO32-4Pin_3.2x2.5mm_HandSoldering
- renumbered J2 to J4
Connections:
- net labels added: AVDD, D_RESET, EN_MIC, PTT, RF_RX, RF_TX, SW_RX, SW_TX
- net labels removed: 3V3
- wire segments 133 -> 171
Other:
- note added: "2.4 GHz / sub-GHz diplexer"
- note added: "38.4 MHz TCXO"
- note added: "Microphone preamplifier"
- moved on the sheet: C14, C15, C21, C23, C24, C25, C30, C33, C35, C36, C37, C40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

Commit message: PCB: Add some part numbers and circuit details
Parts:
- removed C12, C13, C23, C24: TBD, Capacitor_SMD:C_0603_1608Metric_Pad1.05x0.95mm_HandSolder, symbol Device:C
- removed L3, L7: TBD, Inductor_SMD:L_0603_1608Metric_Pad1.05x0.95mm_HandSolder, symbol Device:L
- removed NT1: ~, symbol Device:Net-Tie_2
- removed U1: MCP73831-2-OT, Package_TO_SOT_SMD:SOT-23-5_HandSoldering, symbol Battery_Management:MCP73831-2-OT
- removed U2: MIC5501-3.0YM5, Package_TO_SOT_SMD:SOT-23-5_HandSoldering, symbol Regulator_Linear:MIC5501-3.0YM5
- added C14, C26: 3p, Capacitor_SMD:C_0603_1608Metric_Pad1.05x0.95mm_HandSolder, symbol Device:C
- added C15: 10p, Capacitor_SMD:C_0603_1608Metric_Pad1.05x0.95mm_HandSolder, symbol Device:C
- added C25: 1p, Capacitor_SMD:C_0603_1608Metric_Pad1.05x0.95mm_HandSolder, symbol Device:C
- added C43: 2u2, Capacitor_SMD:C_0603_1608Metric_Pad1.05x0.95mm_HandSolder, symbol Device:C
- added C44, C46: CP, symbol Device:CP
- added C45, C47, C48, C50: 1n, Capacitor_SMD:C_0603_1608Metric_Pad1.05x0.95mm_HandSolder, symbol Device:C
- added C49: 0, Capacitor_SMD:C_0603_1608Metric_Pad1.05x0.95mm_HandSolder, symbol Device:C
- added C5, C9: 100n, Capacitor_SMD:C_0603_1608Metric_Pad1.05x0.95mm_HandSolder, symbol Device:C
- added D2: SM4007PL, Diode_SMD:D_SOD-123F, symbol Device:D
- added FB3, FB4: Ferrite_Bead, Inductor_SMD:L_0603_1608Metric_Pad1.05x0.95mm_HandSolder, symbol Device:Ferrite_Bead
- added J5: SMA, Connector_Coaxial:SMA_Amphenol_901-144_Vertical, symbol Connector:Conn_Coaxial
- added LS1: Speaker, symbol Device:Speaker
- added Q1: FS8205, Package_TO_SOT_SMD:SOT-23-6_Handsoldering, symbol kapula:FS8205
- added Q3, Q4: AO3401A, Package_TO_SOT_SMD:SOT-23_Handsoldering, symbol Transistor_FET:AO3401A
- added R15, R16, R17: 0, Resistor_SMD:R_0603_1608Metric_Pad1.05x0.95mm_HandSolder, symbol Device:R
- added R18, R3: 1k5, Resistor_SMD:R_0603_1608Metric_Pad1.05x0.95mm_HandSolder, symbol Device:R
- added R2: 470, Resistor_SMD:R_0603_1608Metric_Pad1.05x0.95mm_HandSolder, symbol Device:R
- added TP1, TP2, TP3: ~, TestPoint:TestPoint_Pad_2.0x2.0mm, symbol Connector:TestPoint
- added U1: XC6206P332MR, Package_TO_SOT_SMD:SOT-23_Handsoldering, symbol Regulator_Linear:XC6206PxxxMR
- added U2: TP4054, Package_TO_SOT_SMD:SOT-23-5_HandSoldering, symbol kapula:TP4054
- added U3: DW01+G, Package_TO_SOT_SMD:SOT-23-6_Handsoldering, symbol kapula:DW01x
- added U6: LP5907MFX-3.3, Package_TO_SOT_SMD:SOT-23-5_HandSoldering, symbol Regulator_Linear:LP5907MFX-3.3
- added U7: 74HC04D, Package_SO:SOIC-14_3.9x8.7mm_P1.27mm, symbol 74xx:74HC04
- C1, C2, C3, C4: LCSC (none) -> C23630
- C10: renamed from C8; LCSC (none) -> C23630
- C11: renamed from C9; LCSC (none) -> C1588
- C12: renamed from C10; LCSC (none) -> C23630
- C13: renamed from C11; LCSC (none) -> C23630
- C16: renamed from C14; value TBD -> 1p; LCSC (none) -> C23969
- C17: renamed from C15; value TBD -> 1p; LCSC (none) -> C23969
- C18: renamed from C16; LCSC (none) -> C23630
- C19: renamed from C17; LCSC (none) -> C23630
- C20: renamed from C18; LCSC (none) -> C1588
- C21: renamed from C19; LCSC (none) -> C23630
- C22: renamed from C20; LCSC (none) -> C23630
- C24: renamed from C22; LCSC (none) -> C1588
- C27: renamed from C25; value TBD -> 1p; LCSC (none) -> C23969
- C28: renamed from C26; LCSC (none) -> C1588
- C29: renamed from C27; LCSC (none) -> C1588
- C31: renamed from C29; value TBD -> 10p; LCSC (none) -> C1634
- C32: renamed from C30; LCSC (none) -> C1588
- C33: renamed from C31; LCSC (none) -> C23630
- C34: renamed from C32; LCSC (none) -> C1588
- C35: renamed from C33; LCSC (none) -> C23630
- C36: renamed from C34; LCSC (none) -> C1588
- C37: renamed from C35; LCSC (none) -> C23630
- C38: renamed from C36; LCSC (none) -> C1588
- C39: renamed from C37; LCSC (none) -> C14663
- C40: renamed from C38; LCSC (none) -> C1588
- C41: renamed from C39; LCSC (none) -> C1588
- C42: renamed from C40; value 2u2 -> 100n; LCSC (none) -> C14663
- C6: renamed from C5; LCSC (none) -> C14663
- C7: renamed from C6; LCSC (none) -> C14663
- C8: renamed from C7; LCSC (none) -> C14663
- D1: value D -> SM4007PL; footprint (none) -> Diode_SMD:D_SOD-123F; LCSC (none) -> C64898
- L10, L11, L8: value TBD -> 12n; LCSC (none) -> C29258
- L2, L5, L6, L9: value TBD -> 68n; LCSC (none) -> C13415
- L4: value TBD -> 7 mm stub; footprint Inductor_SMD:L_0603_1608Metric_Pad1.05x0.95mm_HandSolder -> NetTie:NetTie-2_SMD_Pad0.5mm
- Q2: renamed from Q1; value BC847 -> MMBT3904; LCSC (none) -> C20526
- R1: value 10k -> 1k5; LCSC (none) -> C22843
- R10: renamed from R8; LCSC (none) -> C21189
- R11: renamed from R9; value 1k -> 470; LCSC (none) -> C23179
- R12: renamed from R10; LCSC (none) -> C25804
- R13: renamed from R11; LCSC (none) -> C25804
- R14: renamed from R12; LCSC (none) -> C25803
- R4: renamed from R2; LCSC (none) -> C21189
- R5: renamed from R3; value 1k -> 470; LCSC (none) -> C23179
- R6: renamed from R4; LCSC (none) -> C21189
- R7: renamed from R5; value 1k -> 470; LCSC (none) -> C23179
- R8: renamed from R6; value 100 -> 470; LCSC (none) -> C23179
- R9: renamed from R7; LCSC (none) -> C21189
- T1, T2: Distributor (none) -> https://www.partco.fi/fi/tarjouseraet/3741-tarmuu-etc4-1-2.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
- U5: renamed from U4; LCSC (none) -> C150894
- X1: value TCO22384001805 -> DSB221SDN; LCSC (none) -> C190737
- renumbered C21 to C23, C28 to C30, U3 to U4
Connections:
- net labels added: BAT-, BC_PROG, BC_VCC, BP_CS, BP_OC, BP_OD, BP_TD, BP_VCC, BiasT, MIC_EN, RX_EN, SPK+, SPK-, SPK_PWM, SPK_VDD, TX_EN, ~CHRG~, ~D_EN~
- net labels removed: EN_MIC, SW_RX, SW_TX
- wire segments 171 -> 256
- no-connect marks 1 -> 0
Other:
- note added: "2.4 GHz / 432 MHz diplexer\nwith Bias-T option"
- note added: "2.4 GHz match to the recommended 23+j7.1 ohm:\n8.4 mm long 0.3 mm wide (50 ohm) trace\n5.6 mm long 0.5 mm wide (37 ohm) open stub"
- note added: "25 ohm to 50 ohm matching lowpass filter\nwith notches near second and third harmonics.\nThe transformer transforms this 25 ohm load\nto 100 ohm differential load\nfor the transmitter output."
- note added: "Battery charger"
- note added: "Battery protection circuit"
- note added: "Connection to a display similar to this:\nhttps://www.ebay.com/itm/133353151886"
- note added: "Input polarity protection"
- note added: "Speaker amplifier\n\nCMOS gate works as a cheap class D output stage.\n32-ohm speaker is recommended."
- note added: "TODO: choose EFR pins"
- note added: "TODO: connector for VCharge"
- note added: "TODO:\nIs the polyfuse useful when there is a protection\ncircuit already? What would be the best place for it?\nHow about battery polarity protection?"
- note added: "User interface"
- note added: "Voltage regulator\n\nPlace of the the two options."
- note removed: "2.4 GHz / sub-GHz diplexer"
- moved on the sheet: BT1, C1, C10, C11, C16, C17, C2, C20, C23, C24, C27, C28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

Commit message: PCB: Attempt some layout for RF parts
Parts:
- removed TP2: ~, TestPoint:TestPoint_Pad_2.0x2.0mm, symbol Connector:TestPoint
- added C34: 10p, Capacitor_SMD:C_0603_1608Metric_Pad1.05x0.95mm_HandSolder, symbol Device:C
- C12: renamed from C11; value 1n -> 220p; LCSC C1588 -> C1603
- C19: renamed from C20; value 1n -> 220p; LCSC C1588 -> C1603
- C22: renamed from C23; footprint Capacitor_SMD:C_0603_1608Metric_Pad1.05x0.95mm_HandSolder -> Capacitor_SMD:C_0402_1005Metric
- C24: value 1n -> 220p; LCSC C1588 -> C1603
- C27: renamed from C48; value 1n -> 220p; LCSC C1588 -> C1603
- C28: renamed from C29; value 1n -> 220p; LCSC C1588 -> C1603
- C29: renamed from C25; value 1p -> 0; DNP (none) -> DNP; LCSC C23969 -> (none)
- C30: renamed from C26; value 3p -> 0; DNP (none) -> DNP; LCSC C46219 -> (none)
- C31: renamed from C28; value 1n -> 220p; LCSC C1588 -> C1603
- C35: renamed from C49; value 0 -> 15p; DNP DNP -> (none)
- C37: renamed from C34; value 1n -> 220p; LCSC C1588 -> C1603
- C38: renamed from C32; value 1n -> 220p; LCSC C1588 -> C1603
- C40: renamed from C36; value 1n -> 220p; LCSC C1588 -> C1603
- C43: renamed from C38; value 1n -> 220p; LCSC C1588 -> C1603
- C46: renamed from C40; value 1n -> 220p; LCSC C1588 -> C1603
- C47: renamed from C45; value 1n -> 220p; LCSC C1588 -> C1603
- C48: renamed from C47; value 1n -> 220p; LCSC C1588 -> C1603
- C49: renamed from C50; value 1n -> 220p; LCSC C1588 -> C1603
- C51: renamed from C41; value 1n -> 220p; LCSC C1588 -> C1603
- J2: renamed from J5; value SMA -> Test; footprint Connector_Coaxial:SMA_Amphenol_901-144_Vertical -> Connector_Coaxial:U.FL_Hirose_U.FL-R-SMT-1_Vertical
- J3: renamed from J1; value SMA -> Test; footprint Connector_Coaxial:SMA_Amphenol_901-144_Vertical -> Connector_Coaxial:U.FL_Hirose_U.FL-R-SMT-1_Vertical
- J5: renamed from J3; value SMA -> Test; footprint Connector_Coaxial:SMA_Amphenol_901-144_Vertical -> Connector_Coaxial:U.FL_Hirose_U.FL-R-SMT-1_Vertical
- L2: renamed from L4; value 7 mm stub -> 6 mm stub
- U6: renamed from U5; footprint Package_TO_SOT_SMD:SOT-363_SC-70-6 -> Package_TO_SOT_SMD:SOT-363_SC-70-6_Handsoldering
- renumbered C42 to C10, C10 to C11, C12 to C13, C13 to C14, C16 to C15, C17 to C16, C18 to C17, C19 to C18, C21 to C20, C22 to C21, C14 to C23, C15 to C25, C27 to C26, C30 to C32, C31 to C33, C33 to C36, C35 to C39, C43 to C41, C37 to C42, C39 to C45, C9 to C5, C46 to C50, C5 to C6, C6 to C7, C7 to C8, C8 to C9, D2 to D1, D1 to D2, J4 to J1, J2 to J4, L5 to L3, L2 to L4, L6 to L5, L8 to L6, L9 to L7, L10 to L8, L11 to L9, Q3 to Q1, Q4 to Q2, Q1 to Q3, Q2 to Q4, R8 to R10, R9 to R11, R10 to R12, R11 to R13, R12 to R14, R13 to R15, R14 to R16, R15 to R17, R16 to R18, R17 to R2, R2 to R3, R3 to R4, R4 to R5, R5 to R6, R6 to R7, R18 to R8, R7 to R9, U6 to U4, U4 to U5
Connections:
- wire segments 256 -> 258
- no-connect marks 0 -> 1
Other:
- moved on the sheet: C29, C30, C35, L8, L9

Commit message: PCB dimensions and more part numbers
Parts:
- added C19: 4u7, Capacitor_SMD:C_0603_1608Metric_Pad1.05x0.95mm_HandSolder, symbol Device:C
- added C42, C46, C5: 15u, Capacitor_Tantalum_SMD:CP_EIA-6032-15_Kemet-U_Pad2.25x2.35mm_HandSolder, symbol Device:CP
- added C6: 220n, Capacitor_SMD:C_0603_1608Metric_Pad1.05x0.95mm_HandSolder, symbol Device:C
- added FB2: GZ2012D601TF, Inductor_SMD:L_0805_2012Metric_Pad1.15x1.40mm_HandSolder, symbol Device:Ferrite_Bead
- added R1: 100k, Resistor_SMD:R_0603_1608Metric_Pad1.05x0.95mm_HandSolder, symbol Device:R
- added R20: 0, Resistor_SMD:R_0603_1608Metric_Pad1.05x0.95mm_HandSolder, symbol Device:R
- added R3: 10k, Resistor_SMD:R_0603_1608Metric_Pad1.05x0.95mm_HandSolder, symbol Device:R
- added TP2: ~, TestPoint:TestPoint_Pad_2.0x2.0mm, symbol Connector:TestPoint
- C1, C2, C3: value 2u2 -> 220n; LCSC C23630 -> C21120
- C10: renamed from C8; value 100n -> 220n; LCSC C14663 -> C21120
- C11: renamed from C9; value 100n -> 220n; LCSC C14663 -> C21120
- C12: renamed from C10; value 100n -> 220n; LCSC C14663 -> C21120
- C13: renamed from C11; value 2u2 -> 4u7; DNP (none) -> DNP; LCSC C23630 -> C19666
- C14: renamed from C12; value 220p -> 220n; LCSC C1603 -> C21120
- C15: renamed from C13; value 2u2 -> 4u7; LCSC C23630 -> C19666
- C16: renamed from C14; value 2u2 -> 4u7; LCSC C23630 -> C19666
- C20: renamed from C17; value 2u2 -> 220n; LCSC C23630 -> C21120
- C21: renamed from C18; value 2u2 -> 220n; LCSC C23630 -> C21120
- C23: renamed from C20; value 2u2 -> 1u; LCSC C23630 -> C15849
- C24: renamed from C21; value 2u2 -> 220n; LCSC C23630 -> C21120
- C37: renamed from C34; LCSC (none) -> C1634
- C38: renamed from C35; LCSC (none) -> C1644
- C39: renamed from C36; value 2u2 -> 4u7; DNP (none) -> DNP; LCSC C23630 -> C19666
- C4: value 2u2 -> 4u7; LCSC C23630 -> C19666
- C40: renamed from C37; value 220p -> 220n; LCSC C1603 -> C21120
- C43: renamed from C39; value 2u2 -> 4u7; LCSC C23630 -> C19666
- C45: renamed from C41; value 2u2 -> 4u7; LCSC C23630 -> C19666
- C47: renamed from C42; value 2u2 -> 4u7; LCSC C23630 -> C19666
- C49: renamed from C44; value CP -> 15u; footprint (none) -> Capacitor_Tantalum_SMD:CP_EIA-6032-15_Kemet-U_Pad2.25x2.35mm_HandSolder
- C50: renamed from C45; value 100n -> 220n; LCSC C14663 -> C21120
- C54: renamed from C50; value CP -> 15u; footprint (none) -> Capacitor_Tantalum_SMD:CP_EIA-6032-15_Kemet-U_Pad2.25x2.35mm_HandSolder
- C56: renamed from C47; DNP DNP -> (none)
- C7: renamed from C5; value 100n -> 220n; LCSC C14663 -> C21120
- C8: renamed from C6; value 100n -> 220n; LCSC C14663 -> C21120
- C9: renamed from C7; value 100n -> 220n; LCSC C14663 -> C21120
- FB1: value Ferrite_Bead -> GZ2012D601TF; footprint Inductor_SMD:L_0603_1608Metric_Pad1.05x0.95mm_HandSolder -> Inductor_SMD:L_0805_2012Metric_Pad1.15x1.40mm_HandSolder; LCSC (none) -> C1017
- FB3: renamed from FB2; value Ferrite_Bead -> GZ2012D601TF; footprint Inductor_SMD:L_0603_1608Metric_Pad1.05x0.95mm_HandSolder -> Inductor_SMD:L_0805_2012Metric_Pad1.15x1.40mm_HandSolder; LCSC (none) -> C1017
- FB4: renamed from FB3; value Ferrite_Bead -> GZ2012D601TF; footprint Inductor_SMD:L_0603_1608Metric_Pad1.05x0.95mm_HandSolder -> Inductor_SMD:L_0805_2012Metric_Pad1.15x1.40mm_HandSolder; LCSC (none) -> C1017
- FB5: renamed from FB4; value Ferrite_Bead -> GZ2012D601TF; footprint Inductor_SMD:L_0603_1608Metric_Pad1.05x0.95mm_HandSolder -> Inductor_SMD:L_0805_2012Metric_Pad1.15x1.40mm_HandSolder; LCSC (none) -> C1017
- L1: footprint Inductor_SMD:L_Taiyo-Yuden_MD-2020 -> Inductor_SMD:L_1206_3216Metric_Pad1.42x1.75mm_HandSolder; LCSC (none) -> C1049
- R12: renamed from R10; value 470 -> 100; LCSC C23179 -> C22775
- R21: renamed from R18; value 0 -> 100; LCSC C21189 -> C22775
- X1: footprint Oscillator:Oscillator_SMD_EuroQuartz_XO32-4Pin_3.2x2.5mm_HandSoldering -> Oscillator:Oscillator_SMD_SeikoEpson_SG210-4Pin_2.5x2.0mm_HandSoldering
- renumbered C15 to C17, C16 to C18, C19 to C22, C22 to C25, C23 to C26, C24 to C27, C25 to C28, C26 to C29, C27 to C30, C28 to C31, C29 to C32, C30 to C33, C31 to C34, C32 to C35, C33 to C36, C38 to C41, C40 to C44, C43 to C48, C46 to C51, C48 to C52, C49 to C53, C51 to C55, R8 to R10, R9 to R11, R11 to R13, R12 to R14, R13 to R15, R14 to R16, R15 to R17, R16 to R18, R17 to R19, R1 to R2, R2 to R4, R3 to R5, R4 to R6, R5 to R7, R6 to R8, R7 to R9
Connections:
- net labels added: RFVDD, VBAT_ADC
- wire segments 258 -> 266
Other:
- note added: "25 ohm to 50 ohm matching lowpass filter\nThe transformer transforms this 25 ohm load\nto 100 ohm differential load\nfor the transmitter output."
- note added: "TODO:\nHow about battery polarity protection?"
- note removed: "25 ohm to 50 ohm matching lowpass filter\nwith notches near second and third harmonics.\nThe transformer transforms this 25 ohm load\nto 100 ohm differential load\nfor the transmitter output."
- note removed: "TODO:\nIs the polyfuse useful when there is a protection\ncircuit already? What would be the best place for it?\nHow about battery polarity protection?"
- moved on the sheet: BT1, C1, C10, C11, C2, C3, C4, C45, C56, C7, C8, C9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

Commit message: PCB: Place components approximately in layout
Parts:
- removed C42, C46, C49, C5, C54: 15u, Capacitor_Tantalum_SMD:CP_EIA-6032-15_Kemet-U_Pad2.25x2.35mm_HandSolder, symbol Device:CP
- added C27: 0, Capacitor_SMD:C_0603_1608Metric_Pad1.05x0.95mm_HandSolder, symbol Device:C
- added C43, C47, C5, C50, C51, C56, C57: 10u, Capacitor_SMD:C_0805_2012Metric_Pad1.15x1.40mm_HandSolder, symbol Device:C
- C4: value 4u7 -> 10u; footprint Capacitor_SMD:C_0603_1608Metric_Pad1.05x0.95mm_HandSolder -> Capacitor_SMD:C_0805_2012Metric_Pad1.15x1.40mm_HandSolder; LCSC C19666 -> C15850
- C44: renamed from C43; value 4u7 -> 220n; LCSC C19666 -> C21120
- C48: renamed from C47; value 4u7 -> 220n; LCSC C19666 -> C21120
- SW1: footprint (none) -> Connector_PinHeader_2.54mm:PinHeader_1x02_P2.54mm_Vertical
- renumbered C27 to C28, C28 to C29, C29 to C30, C30 to C31, C31 to C32, C32 to C33, C33 to C34, C34 to C35, C35 to C36, C36 to C37, C37 to C38, C38 to C39, C39 to C40, C40 to C41, C41 to C42, C44 to C45, C45 to C46, C48 to C49, C50 to C52, C51 to C53, C52 to C54, C53 to C55, C55 to C58, C56 to C59, C7 to C6, C6 to C7, R5 to R2, R2 to R3, R3 to R5
Connections:
- net labels added: PAVDD, RF1_TX
- wire segments 266 -> 277
Other:
- moved on the sheet: C26, C46, C54, C55, C59, FB4, FB5, R12, R19, R20, R21, R6

Commit message: PCB: Most of RF layout routed
Parts:
- removed J2: Test, Connector_Coaxial:U.FL_Hirose_U.FL-R-SMT-1_Vertical, symbol Connector:Conn_Coaxial
- added C15, C49, C6: 220n, Capacitor_SMD:C_0603_1608Metric_Pad1.05x0.95mm_HandSolder, symbol Device:C
- added NT1: ~, NetTie:NetTie-2_SMD_Pad0.5mm, symbol Device:Net-Tie_2
- C16: renamed from C13; value 4u7 -> 220n; DNP DNP -> (none); LCSC C19666 -> C21120
- C44: renamed from C42; value 220p -> 220n; LCSC C1603 -> C21120
- renumbered C9 to C10, C10 to C11, C11 to C12, C12 to C13, C15 to C14, C14 to C17, C16 to C18, C17 to C19, C18 to C20, C19 to C21, C20 to C22, C21 to C23, C22 to C24, C23 to C25, C24 to C26, C25 to C27, C26 to C28, C27 to C29, C28 to C30, C29 to C31, C30 to C32, C31 to C33, C32 to C34, C33 to C35, C34 to C36, C35 to C37, C36 to C38, C37 to C39, C38 to C40, C39 to C41, C40 to C42, C41 to C43, C43 to C45, C44 to C46, C45 to C47, C46 to C48, C47 to C50, C48 to C51, C49 to C52, C50 to C53, C51 to C54, C52 to C55, C53 to C56, C54 to C57, C55 to C58, C56 to C59, C57 to C60, C58 to C61, C59 to C62, C6 to C7, C7 to C8, C8 to C9, J3 to J2, J4 to J3, J5 to J4
Connections:
- wire segments 277 -> 282
Other:
- note added: "17 mm (quarter wave) shorted stub\nto attenuate 2nd harmonic"
- moved on the sheet: C14, C48, FB1

Commit message: PCB: Add some connectors and more routing
Parts:
- removed LS1: Speaker, symbol Device:Speaker
- added C56, C64: ~, Capacitor_SMD:C_0603_1608Metric_Pad1.05x0.95mm_HandSolder, symbol Device:C
- added J1: ~, Connector_PinHeader_2.54mm:PinHeader_1x02_P2.54mm_Vertical, symbol Connector_Generic:Conn_01x02
- added J6: ~, Connector_PinHeader_2.54mm:PinHeader_1x04_P2.54mm_Vertical, symbol Connector_Generic:Conn_01x04
- added J7: ~, Connector_PinHeader_2.54mm:PinHeader_1x06_P2.54mm_Vertical, symbol Connector_Generic:Conn_01x06
- added J8: Conn_01x04_Female, Connector_PinSocket_2.54mm:PinSocket_1x04_P2.54mm_Vertical, symbol Connector:Conn_01x04_Female
- added R22: 0, Resistor_SMD:R_0603_1608Metric_Pad1.05x0.95mm_HandSolder, symbol Device:R
- C17: footprint Capacitor_SMD:C_0603_1608Metric_Pad1.05x0.95mm_HandSolder -> Capacitor_SMD:C_0603_1608Metric
- C62: renamed from C61; DNP DNP -> (none)
- J2: renamed from J1; footprint Connector_PinHeader_2.54mm:PinHeader_1x08_P2.54mm_Vertical -> Connector_PinSocket_2.54mm:PinSocket_1x08_P2.54mm_Vertical
- MK1: footprint Buzzer_Beeper:Buzzer_12x9.5RM7.6 -> Connector_PinHeader_2.54mm:PinHeader_1x02_P2.54mm_Vertical
- SW3: footprint (none) -> Connector_PinHeader_2.54mm:PinHeader_1x02_P2.54mm_Vertical
- TP3: footprint TestPoint:TestPoint_Pad_2.0x2.0mm -> TestPoint:TestPoint_Pad_D1.0mm
- renumbered C57 to C55, C55 to C57, C56 to C58, C58 to C59, C59 to C60, C60 to C61, C62 to C63, J2 to J3, J3 to J4, J4 to J5
Connections:
- net labels added: PA0_TX, PA1_RX, RESET, SPK2+
- net labels removed: RESETn
- wire segments 282 -> 283
- no-connect marks 1 -> 7
Other:
- note added: "SWD\nprogramming connector"
- note added: "Speaker amplifier\n\nCMOS gate works as a cheap class D output stage.\n32-ohm speaker is recommended.\n\nConnect speaker or headphones between SPK+ and SPK-"
- note removed: "Speaker amplifier\n\nCMOS gate works as a cheap class D output stage.\n32-ohm speaker is recommended."
- note removed: "TODO: connector for VCharge"
- moved on the sheet: C55, C63, FB5, R19, R20, R21
