File: kapula/kapula.sch (KiCad schematic (older format))
At the start: 142 parts, among them J2 Display, J3 Test, J4 SMA, J5 Test, J8 Conn_01x04_Female, Q1 AO3401A, Q2 AO3401A, Q3 FS8205, Q4 MMBT3904, SW1 SW_SPST, SW2 EC11B15242B1, SW3 SW_Push, T1 ETC4-1-2TR, T2 ETC4-1-2TR, U1 XC6206P332MR, U2 TP4054, U3 DW01+G, U4 LP5907MFX-3.3, U5 EFR32FG14P233F256GM48-B, U6 AS213-92LF, U7 74HC04D, X1 DSB221SDN

Commit message: PCB: Route display and knob traces
Parts:
- added J6: ~, Connector_PinHeader_2.54mm:PinHeader_1x06_P2.54mm_Vertical, symbol Connector_Generic:Conn_01x06
- added NT2: ~, NetTie:NetTie-2_SMD_Pad0.5mm, symbol Device:Net-Tie_2
- added R13: 100, Resistor_SMD:R_0603_1608Metric_Pad1.05x0.95mm_HandSolder, symbol Device:R
- added R6: 100k, Resistor_SMD:R_0603_1608Metric_Pad1.05x0.95mm_HandSolder, symbol Device:R
- R14: renamed from R12; DNP (none) -> DNP
- renumbered J6 to J8, J8 to J9, R9 to R10, R10 to R11, R11 to R12, R13 to R15, R14 to R16, R15 to R17, R16 to R18, R17 to R19, R18 to R20, R19 to R21, R20 to R22, R21 to R23, R22 to R24, R6 to R7, R7 to R8, R8 to R9
Connections:
- net labels added: PA4, PA5, PB11, PB12, PB13, TCXOGND, TCXO_EN
- wire segments 283 -> 294
- no-connect marks 7 -> 1
Other:
- moved on the sheet: C13, J2, R14, R4
