File: kapula/kapula.sch (KiCad schematic (older format))
At the start: 146 parts, among them J2 Display, J3 Test, J4 SMA, J5 Test, J9 Conn_01x04_Female, Q1 AO3401A, Q2 AO3401A, Q3 FS8205, Q4 MMBT3904, SW1 SW_SPST, SW2 EC11B15242B1, SW3 SW_Push, T1 ETC4-1-2TR, T2 ETC4-1-2TR, U1 XC6206P332MR, U2 TP4054, U3 DW01+G, U4 LP5907MFX-3.3, U5 EFR32FG14P233F256GM48-B, U6 AS213-92LF, U7 74HC04D, X1 DSB221SDN

Commit message: PCB: More layout
Parts:
- removed J6: ~, Connector_PinHeader_2.54mm:PinHeader_1x06_P2.54mm_Vertical, symbol Connector_Generic:Conn_01x06
- added TP10, TP2, TP3, TP4, TP5, TP6, TP7, TP9: ~, TestPoint:TestPoint_Pad_D1.0mm, symbol Connector:TestPoint
- J6: renamed from J7; footprint Connector_PinHeader_2.54mm:PinHeader_1x06_P2.54mm_Vertical -> Connector_PinHeader_2.54mm:PinHeader_1x04_P2.54mm_Vertical; symbol Connector_Generic:Conn_01x06 -> Connector_Generic:Conn_01x04
- renumbered J8 to J7, J9 to J8, TP3 to TP11, TP2 to TP8
Connections:
- wire segments 294 -> 301
- no-connect marks 1 -> 0
Other:
- note removed: "TODO: choose EFR pins"

Commit message: PCB: Everything routed
Parts:
- J7: footprint Connector_PinHeader_2.54mm:PinHeader_1x04_P2.54mm_Vertical -> Connector_PinHeader_2.54mm:PinHeader_1x03_P2.54mm_Vertical; symbol Connector_Generic:Conn_01x04 -> Connector_Generic:Conn_01x03
Connections:
- net labels added: SPKO
Changed lines of the file:
@@
 	9400 9850 9500 9850
 Connection ~ 9500 9850
+Text Label 8100 9350 3    50   ~ 0
+SPK-
 Text Label 8000 9350 3    50   ~ 0
-SPK-
-Text Label 8100 9350 3    50   ~ 0
 SPK+
 Text Label 8200 9350 3    50   ~ 0
 SPK2+
 $Comp
-L Connector_Generic:Conn_01x04 J7
+L Connector_Generic:Conn_01x03 J7
 U 1 1 5F00DC55
 P 8100 9150
 F 0 "J7" V 8018 8862 50  0000 R CNN
 F 1 "~" V 7973 8862 50  0000 R CNN
-F 2 "Connector_PinHeader_2.54mm:PinHeader_1x04_P2.54mm_Vertical" H 8100 9150 50  0001 C CNN
+F 2 "Connector_PinHeader_2.54mm:PinHeader_1x03_P2.54mm_Vertical" H 8100 9150 50  0001 C CNN
 F 3 "~" H 8100 9150 50  0001 C CNN
 	1    8100 9150
@@
 Wire Wire Line
 	2100 1050 2600 1050
-Text Label 8300 9350 3    50   ~ 0
-SPK-
 Text Label 13150 8950 0    50   ~ 0
 RESET
@@
 	-1   0    0    1
 $EndComp
+Text Label 7850 9850 0    50   ~ 0
+SPKO
 $EndSCHEMATC

Commit message: PCB: More clear BOM, some changes
Parts:
- C27, C29, C35, C36, C38: value 0 -> (DNP)
- C42: DNP DNP -> (none)
- C56, C64: value ~ -> (DNP)
- J2: value Display -> ~
- J3, J5: value Test -> U.FL (DNP)
- J8: value Conn_01x04_Female -> ~
- MK1: value Microphone -> ~
- R10, R15: value 0 -> 0 (DNP)
- R14: value 100 -> 100 (DNP)
- SW1: value SW_SPST -> ~
- SW3: value SW_Push -> ~
- U4: value LP5907MFX-3.3 -> LP5907MFX-3.3 (DNP)
