File: hardware_v2/pcb/kapula.kicad_sch (KiCad schematic)
At the start: 166 parts, among them J1 Conn_02x10_Odd_Even, J2 Conn_02x10_Odd_Even, J3 U.FL, J4 U.FL, J5 U.FL, J6 U.FL, Q1 AO3401A, Q1 BSS84, Q2 AO3400A, Q3 AO3400A, Q4 AO3400A, Q5 AO3401A, T1 BW21S7511A01TF, T2 BW21S7511A01TF, T3 BW21S7511A01TF, T4 BW21S7511A01TF, U1 TP4054, U2 DW01+G, U3 XC6206P332MR, U4 FM8002A, U5 EFR32FG14P233F256GM48-B, U6 DSB221SDN, U7 XA213-G4J, Y1 32768 Hz

Commit message: Merge PCB version 2.2
Squashed commit of the following:

commit 29585da15be33afe63cdd15af44b5699f67d3afb
Author: Tatu Peltola <tatu.peltola@gmail.com>
Date:   Wed Feb 21 15:40:03 2024 +0200

    Update documentation for hardware v2.2

commit 29c90c9b898eb7544d7174a70b0680bc57b382f8
Author: Tatu Peltola <tatu.peltola@gmail.com>
Date:   Tue Feb 20 14:58:30 2024 +0200

    PCB: Rename net 1V8 to DVDD

commit e3e53bd1db9ca6e578998accadfb8cad49b924a5
Author: Tatu Peltola <tatu.peltola@gmail.com>
Date:   Fri Jan 26 21:21:14 2024 +0200

    PCB: Add information on ordering

commit 15d7fdc716a4f514bde473c7c7c42e8fd8a06f95
Author: Tatu Peltola <tatu.peltola@gmail.com>
Date:   Fri Jan 26 20:24:04 2024 +0200

    PCB: Cleanup layout around TCXO

commit 6a4db70d40617c021f0c2f35424b09177388460d
Author: Tatu Peltola <tatu.peltola@gmail.com>
Date:   Fri Jan 26 20:05:08 2024 +0200

    PCB: Change some RF matching footprints, improve silkscreen

commit c4c77dd10fb55911e6db8f7eeaab550065731a89
Author: Tatu Peltola <tatu.peltola@gmail.com>
Date:   Wed Jan 24 17:45:02 2024 +0200

    PCB: Commit some changes

commit d3d1ba59bc8299044051a8e6796e96fdff23bdfd
Author: Tatu Peltola <tatu.peltola@gmail.com>
Date:   Thu Jan 18 20:50:07 2024 +0200

    PCB: Refill zones after moving connectors

commit e68e224a804bc1105053c6d5c5337a184e776e7c
Author: Tatu Peltola <tatu.peltola@gmail.com>
Date:   Thu Jan 18 20:46:27 2024 +0200

    PCB: Move connectors exactly to grid

commit 831c9cb543746d85673284f06b40a8616ee1c0ab
Author: Tatu Peltola <tatu.peltola@gmail.com>
Date:   Thu Jan 11 15:46:53 2024 +0200

    PCB: Fix some silkscreen texts

commit 53a4e8818c62c7af800c843000d9c5c4781ee048
Author: Tatu Peltola <tatu.peltola@gmail.com>
Date:   Thu Jan 11 01:13:23 2024 +0200

    PCB: Route TCXO again

commit a34db1df76e42d1f0f01b91663b2ec0ce728b371
Author: Tatu Peltola <tatu.peltola@gmail.com>
Date:   Thu Jan 11 00:56:23 2024 +0200

    PCB: Make some space for TCXO again

commit 3292631f53a83882c25395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
Parts:
- removed J8: ~, Connector_PinSocket_2.54mm:PinSocket_1x04_P2.54mm_Vertical, symbol Connector:Conn_01x04_Socket
- added R24: 1M, Resistor_SMD:R_0402_1005Metric, symbol Device:R
- C15: footprint kapula:C_0402_to_0603_HandSolder -> Capacitor_SMD:C_0402_1005Metric_Pad0.74x0.62mm_HandSolder
- C74, C82: footprint kapula:C_0402_to_0603_HandSolder -> Capacitor_SMD:C_0603_1608Metric_Pad1.08x0.95mm_HandSolder; LCSC C1523 -> C1588
- C83, C84, C85: footprint kapula:C_0402_to_0603_HandSolder -> Capacitor_SMD:C_0603_1608Metric_Pad1.08x0.95mm_HandSolder
- J7: footprint kapula:DZ127S-22-10-55 -> Connector_PinHeader_2.54mm:PinHeader_2x05_P2.54mm_Vertical; LCSC C5160761 -> (none)
- L71, L72, L74, L75, L76, L77: footprint kapula:L_0402_to_0603_HandSolder -> Inductor_SMD:L_0402_1005Metric_Pad0.77x0.64mm_HandSolder
- R1, R13: footprint Resistor_SMD:R_0402_1005Metric -> Resistor_SMD:R_0603_1608Metric_Pad0.98x0.95mm_HandSolder; LCSC C17168 -> C21189
- R11, R12: footprint kapula:R_0402_to_0603_HandSolder -> Resistor_SMD:R_0402_1005Metric_Pad0.72x0.64mm_HandSolder
- R16: value 1M -> 330k; LCSC C26083 -> C25778
- R18: footprint Resistor_SMD:R_0402_1005Metric -> Resistor_SMD:R_0603_1608Metric_Pad0.98x0.95mm_HandSolder; LCSC C25768 -> C31850
- R19: value 22k -> 47k; footprint Resistor_SMD:R_0402_1005Metric -> Resistor_SMD:R_0603_1608Metric_Pad0.98x0.95mm_HandSolder; LCSC C25768 -> C25819
- R2, R33, R34: footprint kapula:R_0402_to_0603_HandSolder -> Resistor_SMD:R_0603_1608Metric_Pad0.98x0.95mm_HandSolder
- R35, R44, R45, R46, R47, R48, R5, R78: footprint kapula:R_0402_to_0603_HandSolder -> Resistor_SMD:R_0603_1608Metric_Pad0.98x0.95mm_HandSolder; LCSC C17168 -> C21189
- R4: footprint kapula:R_0402_to_0603_HandSolder -> Resistor_SMD:R_0603_1608Metric
- U6: value DSB221SDN -> TG2016SMN 38.4000M-MCGNNM3
Connections:
- net GND: now also R24.1; no longer J2.7 (Pin_7)
- net RX_EN_SW: now also C81.1, U7.4 (V2); no longer C80.1, U7.6 (V1)
- net TX_EN_SW: now also C80.1, U7.6 (V1); no longer C81.1, U7.4 (V2)
- net VOL_Out: now also R24.2
- net 1V8 renamed DVDD
- net DVDD: now also J2.7 (Pin_7)
Other:
- note added: "0.2 mm wide 6 mm stub"
- note added: "SWD programming connector"
- note removed: "0.2 mm wide 7 mm stub"
- note removed: "Two alternative SWD programming connectors"
- moved on the sheet: C12, C13, C14, C15, R14, R76, R77
